File: designs/Biofilms_PCB/routing_board.sch (KiCad schematic (older format))
At the start: 16 parts, among them J1 Arduino TL, J10 DC PWR, J11 Arduino IO, J12 Arduino Power Out, J2 Arduino BL, J3 Motor Power, J4 Arduino TR, J5 Arduino BR, J6 Servo, J7 Limit Switch, J8 Motor Driver, J9 Solenoid, Q1 Q_NPN_Darlington_BCE

Commit message: finalized v2 of biofilms PCB
Parts:
- removed J11: Arduino IO, Socket_Strips:Socket_Strip_Straight_1x12_Pitch2.54mm, symbol Conn_01x12
- added D1, D3, D4, D5, D6, D7, D8, D9: LED, LEDs:LED_0603_HandSoldering, symbol LED
- added J11: Analog In, Pin_Headers:Pin_Header_Straight_1x06_Pitch2.54mm, symbol Conn_01x06
- added J13: Digital Out, Pin_Headers:Pin_Header_Straight_1x06_Pitch2.54mm, symbol Conn_01x06
- added Q2: Q_PNP_BEC, TO_SOT_Packages_SMD:SOT-23, symbol Q_PNP_BEC
- added R1, R10, R3, R4, R5, R6, R7, R8: 2.5k, Resistors_SMD:R_0603_HandSoldering, symbol R
- added R9: 150k, Resistors_SMD:R_0603_HandSoldering, symbol R
- D2: renamed from D1; footprint (none) -> Diodes_SMD:D_SOD-123F
- J9: renamed from J12; footprint (none) -> Pin_Headers:Pin_Header_Straight_1x04_Pitch2.54mm
- Q1: footprint (none) -> TO_SOT_Packages_SMD:SOT-23
- R2: renamed from R1; value 10k -> 150k; footprint (none) -> Resistors_SMD:R_0603_HandSoldering
- S1: footprint (none) -> Buttons_Switches_SMD:SW_DIP_x3_W8.61mm_Slide_LowProfile
- renumbered J9 to J10, J10 to J12, J8 to J7, J7 to J8
Connections:
- net +12V: now also R1.2, R3.2
- net AI0: now also J11.1 (Pin_1)
- net AI1: now also J11.2 (Pin_2)
- net AI2: now also J11.3 (Pin_3)
- net AI3: now also J11.4 (Pin_4)
- net AI4: now also J11.5 (Pin_5)
- net AI5: now also J11.6 (Pin_6)
- net DO0: now also J13.1 (Pin_1), R4.2
- net DO1: now also J13.2 (Pin_2), R5.2
- net DO2: now also J13.3 (Pin_3), R6.2
- net DO3: now also J13.4 (Pin_4), R7.2
- net DO4: now also J13.5 (Pin_5), R8.2
- net ENABLE: now also R9.2
- net GND: now also D1.1 (K), D4.1 (K), D5.1 (K), D6.1 (K), D7.1 (K), D8.1 (K), J13.6 (Pin_6), R10.1
- net MC_5V: now reaches J7.4 (Pin_4)
- net MC_5V: now also Q2.2 (E)
- net at D2.2 (A), J10.1 (Pin_1), Q1.2 (C): now also D3.1 (K)
- new net: D4.2 (A), R4.1
- new net: D5.2 (A), R5.1
- new net: D6.2 (A), R6.1
- new net: D7.2 (A), R7.1
- new net: D8.2 (A), R8.1
- new net: D3.2 (A), R3.1
- new net: D9.1 (K), R10.2
- new net: D9.2 (A), Q2.3 (C)
- new net: Q2.1 (B), R9.1
- new net: D1.2 (A), R1.1
- no-connect marks 11 -> 10
Other:
- moved on the sheet: J7, J9
