File: designs/CapperDecapper/KiCAD 5/Capper Decapper/Capper Decapper.sch (KiCad schematic (older format))
At the start: 50 parts, among them J1 Screw_Terminal_01x02, J2 Conn_01x03_Female, J3 Analog_Zero, J4 Pi_Signals, J5 Motor_Power, U1 L2293, U10 INA214, U11 L2293, U12 INA214, U13 INA214, U2 INA214, U3 INA214, U4 L2293, U5 INA214, U6 INA214, U7 ADP172, U8 L2293, U9 INA214

Commit message: complete 1st draft of capper/decapper PCB
Parts:
- removed R?: R_US, symbol Device:R_US
- added C17: C, Capacitor_SMD:C_0603_1608Metric, symbol Device:C
- Q1: renamed from Q?; footprint (none) -> Package_TO_SOT_SMD:SOT-23
- R3: renamed from R?; footprint (none) -> Resistor_SMD:R_0603_1608Metric
- RV1: renamed from RV?; footprint (none) -> CustomFootprints:R_TRIM_4mm_Gull
- U14: renamed from U?; value LM1084-ADJ -> LM338-ADJ; footprint (none) -> Package_TO_SOT_THT:TO-220-3_Vertical
Connections:
- wire segments 269 -> 272

Commit message: PWM capper decapper board
Parts:
- removed C6: C, Capacitor_SMD:C_0603_1608Metric, symbol Device:C
- removed J2: Conn_01x03_Female, Connector_PinSocket_2.54mm:PinSocket_1x03_P2.54mm_Horizontal, symbol Connector:Conn_01x03_Female
- removed J3: Analog_Zero, Connector_PinSocket_2.54mm:PinSocket_1x11_P2.54mm_Vertical, symbol Connector:Conn_01x11_Female
- removed J4: Pi_Signals, Connector_PinSocket_2.54mm:PinSocket_1x20_P2.54mm_Vertical, symbol Connector:Conn_01x20_Female
- removed RV1: R_POT, CustomFootprints:R_TRIM_4mm_Gull, symbol Device:R_POT
- removed U14: LM338-ADJ, Package_TO_SOT_THT:TO-220-3_Vertical, symbol Regulator_Linear:LM1084-ADJ
- removed U7: ADP172, Package_BGA:WLP-4_0.86x0.86mm_P0.4mm, symbol CustomComponents:ADP172
- added C10, C14, C15, C22, C23, C4, C5: 22nF, Capacitor_SMD:C_0603_1608Metric, symbol Device:C
- added C25: 33uF, Capacitor_SMD:C_0603_1608Metric, symbol Device:C
- added J1: Pi Control Signals, Connector_PinSocket_2.54mm:PinSocket_1x24_P2.54mm_Vertical, symbol Connector:Conn_01x24_Female
- added L1: L_Coupled, Inductor_THT:L_CommonMode_Wuerth_WE-CMB-S, symbol Device:L_Coupled
- added PS1: R-7XX, Resistor_THT:R_Array_SIP12, symbol CustomComponents:R-7XX
- added R10, R14, R15, R18, R5, R6, R9: 20k, Resistor_SMD:R_0603_1608Metric, symbol Device:R_US
- added R19: 20K, Resistor_SMD:R_0603_1608Metric, symbol Device:R_US
- added U11: V7805-1500R, Package_SIP:SIP3_11.6x8.5mm, symbol Regulator_Switching:R-78B9.0-2.0
- added U14: MAX6018BEUR16, Package_TO_SOT_SMD:SOT-23, symbol Regulator_Linear:APE8865NR-17-HF-3
- C1, C11: value C -> 0.01uF
- C12, C13, C3: value C -> 0.1uF
- C17: value C -> 33uF
- C18: renamed from C14; value C -> 0.01uF
- C19: renamed from C8; value C -> 0.1uF
- C2: value C -> 0.1uF; Spice_Model (none) -> 0.01u; Spice_Netlist_Enabled (none) -> Y; Spice_Primitive (none) -> C
- C20: renamed from C15; value C -> 0.1uF
- C21: renamed from C16; value C -> 0.1uF
- C24: renamed from C10; value C -> 0.01uF
- C6: renamed from C4; value C -> 0.1uF
- C7: renamed from C5; value C -> 0.01uF
- C8: renamed from C7; value C -> 0.1uF
- C9: value C -> 22nF
- D1: value D_Schottky_Small_ALT -> Schottky
- J3: renamed from J1; value Screw_Terminal_01x02 -> Screw_Term
- R1: renamed from R8; value R_US -> 330R
- R11: renamed from R3; value R_US -> 5k
- R12: renamed from R6; value R_US -> 0.05R
- R13: renamed from R7; value R_US -> 0.05R
- R16: renamed from R10; value R_US -> 0.05R
- R17: renamed from R11; value R_US -> 0.05R
- R2: renamed from R9; value R_US -> 330R
- R3: renamed from R1; value R_US -> 0.05R; Spice_Model (none) -> 50mR; Spice_Netlist_Enabled (none) -> Y; Spice_Primitive (none) -> R
- R4: renamed from R2; value R_US -> 0.05R
- R7: renamed from R4; value R_US -> 0.05R
- R8: renamed from R5; value R_US -> 0.05R
- U2: Spice_Lib_File (none) -> /Users/robert.puccinelli/Downloads/INA214_PSPICE_AIO/INA214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; Spice_Model (none) -> pulse(0 50m 1u 1u 1u 25u 50u); Spice_Netlist_Enabled (none) -> Y; Spice_Primitive (none) -> I
- renumbered J5 to J2, U11 to U10, U8 to U7, U9 to U8, U10 to U9
Connections:
- net labels added: EN1, EN2, EN3, EN4, EN5, EN6, EN7, EN8, FWD, REV, VBUS
- net labels removed: +36V, MOT1_FWD, MOT1_REV, MOT2_FWD, MOT2_REV, MOT3_FWD, MOT3_REV, MOT4_FWD, MOT4_REV, MOT5_FWD, MOT5_REV, MOT6_FWD, MOT6_REV, MOT7_FWD, MOT7_REV, MOT8_FWD, MOT8_REV
- wire segments 272 -> 311
- no-connect marks 0 -> 1
Other:
- note added: "18V"
- note added: "Motor 9V"
- note removed: "36V"
- note removed: "Analog Zero"
- note removed: "V_motor"

Commit message: Capper/Decapper HW Control Board Rev A
Parts:
- removed C1, C11, C18: 0.01uF, Capacitor_SMD:C_0603_1608Metric, symbol Device:C
- removed C10, C5: 22nF, Capacitor_SMD:C_0603_1608Metric, symbol Device:C
- removed C17, C25: 33uF, Capacitor_SMD:C_0603_1608Metric, symbol Device:C
- removed C2, C20, C21: 0.1uF, Capacitor_SMD:C_0603_1608Metric, symbol Device:C
- removed L1: L_Coupled, Inductor_THT:L_CommonMode_Wuerth_WE-CMB-S, symbol Device:L_Coupled
- removed PS1: R-7XX, Resistor_THT:R_Array_SIP12, symbol CustomComponents:R-7XX
- removed R3: 0.05R, Resistor_SMD:R_1206_3216Metric, symbol Device:R_US
- removed U1, U10, U4, U7: L2293, Package_QFP:LQFP-32-1EP_5x5mm_P0.5mm_EP3.45x3.45mm, symbol CustomComponents:L2293
- removed U2, U6: INA214, Package_TO_SOT_SMD:SOT-363_SC-70-6, symbol CustomComponents:INA214
- added C10, C16, C25, C4: 2.2uF, Capacitor_SMD:C_0603_1608Metric, symbol Device:C_Small
- added C11, C18, C27, C5: 10nF, Capacitor_SMD:C_0603_1608Metric, symbol Device:C_Small
- added C17, C20, C30, C31, C32, C33: 10uF, Capacitor_Tantalum_SMD:CP_EIA-3528-12_Kemet-T, symbol Device:CP_Small
- added C19, C28, C29: 0.1uF, Capacitor_SMD:C_0603_1608Metric, symbol Device:C
- added C24, C3: 22nF, Capacitor_SMD:C_0603_1608Metric, symbol Device:C
- added C34, C35, C36, C37: 0.1uF, Capacitor_SMD:C_0603_1608Metric, symbol Device:C_Small
- added D2: Schottky, Diode_SMD:D_SMA, symbol Device:D_Schottky_Small_ALT
- added L1: 22uH, Inductor_SMD:L_Wuerth_HCI-1365, symbol Device:L_Small
- added MH1, MH2: MountingHole, MountingHole:MountingHole_3mm, symbol Mechanical:MountingHole
- added R20: 14.2K, Resistor_SMD:R_0603_1608Metric, symbol Device:R_US
- added R21: 2K, Resistor_SMD:R_0603_1608Metric, symbol Device:R_US
- added R5: 20k, Resistor_SMD:R_0603_1608Metric, symbol Device:R_US
- added U10, U15, U2, U6: 74AHC08, Package_DFN_QFN:Texas_S-PVQFN-N14_ThermalVias, symbol CustomComponents:74AHC08
- added U11, U16, U3, U7: DRV8833RTY, Package_DFN_QFN:WQFN-16-1EP_4x4mm_P0.65mm_EP2.1x2.1mm, symbol Driver_Motor:DRV8833RTY
- added U18, U4: INA214, Package_TO_SOT_SMD:SOT-363_SC-70-6, symbol CustomComponents:INA214
- added U19: AP1501A, Package_TO_SOT_SMD:TO-263-5_TabPin3, symbol CustomComponents:AP1501A
- C13: value 0.1uF -> 22nF
- C14, C23: value 22nF -> 0.1uF
- C21: renamed from C19; value 0.1uF -> 0.33uF
- C7: value 0.01uF -> 22nF
- Q1: value Q_NMOS_GDS -> Q_NMOS_GSD; symbol Device:Q_NMOS_GDS -> Device:Q_NMOS_GSD
- R10, R15, R6: value 20k -> 0.05R; footprint Resistor_SMD:R_0603_1608Metric -> Resistor_SMD:R_1206_3216Metric
- R13, R17, R8: value 0.05R -> 20k; footprint Resistor_SMD:R_1206_3216Metric -> Resistor_SMD:R_0603_1608Metric
- R19: value 20K -> 0.05R; footprint Resistor_SMD:R_0603_1608Metric -> Resistor_SMD:R_1206_3216Metric
- U14: renamed from U11; footprint Package_SIP:SIP3_11.6x8.5mm -> Package_TO_SOT_SMD:TO-252-3_TabPin2; symbol Regulator_Switching:R-78B9.0-2.0 -> Regulator_Linear:L7805
- renumbered C4 to C1, C3 to C2, C24 to C26, R4 to R1, R5 to R2, R1 to R3, R2 to R4, U3 to U1, U14 to U17
Connections:
- wire segments 311 -> 396
- no-connect marks 1 -> 4
Other:
- moved on the sheet: U17

Commit message: AND gate updated, ordered
Parts:
- U10, U15, U2, U6: footprint Package_DFN_QFN:Texas_S-PVQFN-N14_ThermalVias -> CustomFootprints:PVQFN-14
- U14: value V7805-1500R -> L7805
Changed lines of the file:
@@
 P 9400 5300
 F 0 "U14" H 9400 5542 50  0000 C CNN
-F 1 "V7805-1500R" H 9400 5451 50  0000 C CNN
+F 1 "L7805" H 9400 5451 50  0000 C CNN
 F 2 "Package_TO_SOT_SMD:TO-252-3_TabPin2" H 9450 5050 50  0001 L CIN
 F 3 "https://www.recom-power.com/pdf/Innoline/R-78Bxx-2.0.pdf" H 9400 5300 50  0001 C CNN
@@
 F 0 "U15" H 10341 1646 50  0000 L CNN
 F 1 "74AHC08" H 10341 1555 50  0000 L CNN
-F 2 "Package_DFN_QFN:Texas_S-PVQFN-N14_ThermalVias" H 10300 1050 50  0001 C CNN
+F 2 "CustomFootprints:PVQFN-14" H 10300 1050 50  0001 C CNN
 F 3 "" H 10300 1050 50  0001 C CNN
 	1    9700 1600
@@
 F 0 "U10" H 7691 1696 50  0000 L CNN
 F 1 "74AHC08" H 7691 1605 50  0000 L CNN
-F 2 "Package_DFN_QFN:Texas_S-PVQFN-N14_ThermalVias" H 7650 1100 50  0001 C CNN
+F 2 "CustomFootprints:PVQFN-14" H 7650 1100 50  0001 C CNN
 F 3 "" H 7650 1100 50  0001 C CNN
 	1    7050 1650
@@
 F 0 "U6" H 5091 1646 50  0000 L CNN
 F 1 "74AHC08" H 5091 1555 50  0000 L CNN
-F 2 "Package_DFN_QFN:Texas_S-PVQFN-N14_ThermalVias" H 5050 1050 50  0001 C CNN
+F 2 "CustomFootprints:PVQFN-14" H 5050 1050 50  0001 C CNN
 F 3 "" H 5050 1050 50  0001 C CNN
 	1    4450 1600
@@
 F 0 "U2" H 1209 1646 50  0000 R CNN
 F 1 "74AHC08" H 1209 1555 50  0000 R CNN
-F 2 "Package_DFN_QFN:Texas_S-PVQFN-N14_ThermalVias" H 2450 1050 50  0001 C CNN
+F 2 "CustomFootprints:PVQFN-14" H 2450 1050 50  0001 C CNN
 F 3 "" H 2450 1050 50  0001 C CNN
 	1    1850 1600

Commit message: Directory update
Parts:
- removed Q1: Q_NMOS_GSD, Package_TO_SOT_SMD:SOT-23, symbol Device:Q_NMOS_GSD
- removed R11: 5k, Resistor_SMD:R_0603_1608Metric, symbol Device:R_US
- added Q?: Q_PMOS_GSD, symbol Device:Q_PMOS_GSD
- added R? (x2): R_US, symbol Device:R_US
Connections:
- wire segments 396 -> 391
Changed lines of the file:
@@
 L Device:D_Schottky_Small_ALT D1
 U 1 1 5BB16426
-P 7000 5850
-F 0 "D1" V 7046 5782 50  0000 R CNN
-F 1 "Schottky" V 7200 5800 50  0000 R CNN
-F 2 "Diode_SMD:D_SMA" V 7000 5850 50  0001 C CNN
-F 3 "~" V 7000 5850 50  0001 C CNN
-	1    7000 5850
-	0    1    1    0
-$EndComp
-Text Label 6000 5800 2    50   ~ 0
+P 6400 6300
+F 0 "D1" V 6500 6500 50  0000 R CNN
+F 1 "Schottky" V 6400 6700 50  0000 R CNN
+F 2 "Diode_SMD:D_SMA" V 6400 6300 50  0001 C CNN
+F 3 "~" V 6400 6300 50  0001 C CNN
+	1    6400 6300
+	0    1    1    0
+$EndComp
+Text Label 6000 5850 2    50   ~ 0
 SOLSET
 Wire Wire Line
 	5650 5800 5650 6400
-Text Label 6700 5450 0    50   ~ 0
+Text Label 6450 6100 0    50   ~ 0
 SOL+
 $Comp
@@
 Text Label 1600 4000 0    50   ~ 0
 5V
-$Comp
-L Device:Q_NMOS_GSD Q1
-U 1 1 5B9EE045
-P 6500 5800
-F 0 "Q1" H 6705 5846 50  0000 L CNN
-F 1 "Q_NMOS_GSD" H 6100 5950 50  0000 L CNN
-F 2 "Package_TO_SOT_SMD:SOT-23" H 6700 5900 50  0001 C CNN
-F 3 "~" H 6500 5800 50  0001 C CNN
-	1    6500 5800
-	1    0    0    -1
-$EndComp
-Wire Wire Line
-	6600 5450 6700 5450
-Wire Wire Line
-	6600 5600 6600 5550
 Wire Wire Line
 	5650 5700 5650 5300
-Connection ~ 6600 6400
-$Comp
-L Device:R_US R11
-U 1 1 5BBBD34E
-P 6050 5950
-F 0 "R11" H 5982 5904 50  0000 R CNN
-F 1 "5k" H 5982 5995 50  0000 R CNN
-F 2 "Resistor_SMD:R_0603_1608Metric" V 6090 5940 50  0001 C CNN
-F 3 "~" H 6050 5950 50  0001 C CNN
-	1    6050 5950
-	-1   0    0    1
-$EndComp
-Wire Wire Line
-	6050 6100 6050 6400
-Wire Wire Line
-	6000 5800 6050 5800
-Connection ~ 6050 5800
-Wire Wire Line
-	6050 5800 6300 5800
-Connection ~ 6050 6400
-Wire Wire Line
-	6050 6400 5650 6400
-Wire Wire Line
-	6050 6400 6600 6400
 $Comp
 L power:GND #PWR04
@@
 	1    0    0    -1
 $EndComp
-Wire Wire Line
-	5650 5300 6600 5300
-Connection ~ 6600 5300
 Text Label 2250 6400 2    50   ~ 0
 FWD
@@
 Wire Wire Line
 	8300 6050 8300 6400
-Wire Wire Line
-	6600 5300 7650 5300
-Wire Wire Line
-	6600 6400 7000 6400
 Connection ~ 8300 6400
 Wire Wire Line
@@
 $EndComp
 Connection ~ 3000 3200
-Connection ~ 6600 5450
-Wire Wire Line
-	6600 5450 6600 5300
-Wire Wire Line
-	6600 6000 6600 6400
-Wire Wire Line
-	7000 5950 7000 6400
-Connection ~ 7000 6400
-Wire Wire Line
-	7000 6400 7300 6400
-Wire Wire Line
-	7000 5750 7000 5550
-Wire Wire Line
-	7000 5550 6600 5550
-Connection ~ 6600 5550
-Wire Wire Line
-	6600 5550 6600 5450
 Text Label 8000 6250 0    50   ~ 0
 V_motor
@@
 Wire Wire Line
 	7950 6100 7950 6250
+$Comp
+L Device:R_US R?
+U 1 1 5C74585C
+P 6100 5550
+F 0 "R?" H 6032 5504 50  0000 R CNN
+F 1 "R_US" H 6032 5595 50  0000 R CNN
+F 2 "" V 6140 5540 50  0001 C CNN
+F 3 "~" H 6100 5550 50  0001 C CNN
+	1    6100 5550
+	-1   0    0    1
+$EndComp
+Wire Wire Line
+	6100 5700 6100 5850
+$Comp
+L Device:R_US R?
+U 1 1 5C76DF81
+P 6400 5450
+F 0 "R?" H 6468 5496 50  0000 L CNN
+F 1 "R_US" H 6468 5405 50  0000 L CNN
+F 2 "" V 6440 5440 50  0001 C CNN
+F 3 "~" H 6400 5450 50  0001 C CNN
+	1    6400 5450
+	1    0    0    -1
+$EndComp
+Wire Wire Line
+	6000 5850 6100 5850
+Wire Wire Line
+	5650 5300 6100 5300
+Connection ~ 6400 5300
+Wire Wire Line
+	6400 5300 7650 5300
+Wire Wire Line
+	6400 5600 6400 5650
+Wire Wire Line
+	6100 5400 6100 5300
+Connection ~ 6100 5300
+Wire Wire Line
+	6100 5300 6400 5300
+Wire Wire Line
+	6400 6050 6400 6100
+Wire Wire Line
+	5650 6400 6400 6400
+Connection ~ 6400 6400
+Wire Wire Line
+	6400 6400 7300 6400
+Wire Wire Line
+	6400 6100 6450 6100
+Connection ~ 6400 6100
+Wire Wire Line
+	6400 6100 6400 6200
+$Comp
+L Device:Q_PMOS_GSD Q?
+U 1 1 5CB67504
+P 6300 5850
+F 0 "Q?" H 6506 5896 50  0000 L CNN
+F 1 "Q_PMOS_GSD" H 6506 5805 50  0000 L CNN
+F 2 "" H 6500 5950 50  0001 C CNN
+F 3 "~" H 6300 5850 50  0001 C CNN
+	1    6300 5850
+	1    0    0    -1
+$EndComp
+Connection ~ 6100 5850
 $EndSCHEMATC
