File: designs/CapperDecapper/Capper Decapper v2/MotorDriverBoard_v2.sch (KiCad schematic (older format))
At the start: 115 parts, among them J1 Stepper_I2C, J2 Power_Connector, J3 Solenoid_Connector, J4 Pi_Header, J5 DC_Connector, J6 Stepper_I2C, J7 Toggle_Connector, J8 Run_Connector, J9 Pause_Connector, Q1 Q_NMOS_GSD, Q10 Q_NMOS_GSD, Q11 Q_NMOS_GSD, Q12 Q_NMOS_GSD, Q13 Q_NMOS_GSD, Q14 Q_NMOS_GSD, Q15 Q_NMOS_GSD, Q16 Q_NMOS_GSD, Q17 Q_NMOS_GSD, Q2 Q_NMOS_GSD, Q3 Q_NMOS_GSD, Q4 Q_NMOS_GSD, Q5 Q_NMOS_GSD, Q6 Q_NMOS_GSD, Q7 Q_NMOS_GSD, Q8 Q_NMOS_GSD, Q9 Q_NMOS_GSD, U1 DRV8833RTY, U10 74LVC2G14, U11 AP6503, U12 AP6503, U2 DRV8833RTY, U3 DRV8833RTY, U4 DRV8833RTY, U5 MCP3008, U6 CBT3245A, U7 CBT3245A, U8 INA4180, U9 INA4180

Commit message: Capper Decapper REV B on OSHPark
Parts:
- added C30, C31: 100nF, Capacitor_SMD:C_0603_1608Metric, symbol Device:C
- added H1, H2, H3: MountingHole, MountingHole:MountingHole_2.2mm_M2, symbol Mechanical:MountingHole
- added R32: 5k, Resistor_SMD:R_0603_1608Metric, symbol Device:R
- added TP1: InvPwmF, TestPoint:TestPoint_Pad_D1.0mm, symbol Connector:TestPoint
- added TP2: InvPwmR, TestPoint:TestPoint_Pad_D1.0mm, symbol Connector:TestPoint
- added TP3: 2Fwd, TestPoint:TestPoint_Pad_D1.0mm, symbol Connector:TestPoint
- added TP4: 2Rev, TestPoint:TestPoint_Pad_D1.0mm, symbol Connector:TestPoint
- added U13: TXB0102DCU, Package_SO:VSSOP-8_2.4x2.1mm_P0.5mm, symbol Logic_LevelTranslator:TXB0102DCU
- C20: footprint Capacitor_SMD:C_0603_1608Metric -> Capacitor_SMD:C_0805_2012Metric
- R10, R11, R12, R5, R6, R7, R8, R9: value 47m -> 50m; footprint Resistor_SMD:R_0603_1608Metric -> Resistor_SMD:R_1206_3216Metric
Connections:
- net +3V3: now also C30.1, R32.2, U13.3 (VCCA)
- net +5V: now also C31.2, U13.7 (VCCB)
- net GND: now also J5.13 (Pin_13), J5.14 (Pin_14), J5.18 (Pin_18), J5.19 (Pin_19), C30.2, C31.1, U13.2 (GND)
- net InvFwd: now also TP1.1
- net InvRev: now also TP2.1
- net Mot2Fwd: now also TP3.1
- net Mot2Rev: now also TP4.1
- net SCL: now also U13.4 (A2); no longer J1.3 (Pin_3), J6.3 (Pin_3)
- net SDA: now also U13.5 (A1); no longer J1.2 (Pin_2), J6.2 (Pin_2)
- new net: J1.3 (Pin_3), J6.3 (Pin_3), U13.1 (B2)
- new net: R32.1, U13.6 (OE)
- new net: J1.2 (Pin_2), J6.2 (Pin_2), U13.8 (B1)
- no-connect marks 13 -> 9
Other:
- note added: "Bulk Connectors"
- note added: "DC Motor Components"
- note added: "Peripherals"
- note added: "Power Regulation"
- moved on the sheet: C1, C10, C11, C12, C13, C14, C15, C16, C17, C18, C19, C2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
