File: designs/CapperDecapper/Capper Decapper v2/MotorDriverBoard_v2.sch (KiCad schematic (older format))
At the start: 126 parts, among them J1 Stepper_I2C, J2 Power_Connector, J3 Solenoid_Connector, J4 Pi_Header, J5 DC_Connector, J6 Stepper_I2C, J7 Toggle_Connector, J8 Run_Connector, J9 Pause_Connector, Q1 Q_NMOS_GSD, Q10 Q_NMOS_GSD, Q11 Q_NMOS_GSD, Q12 Q_NMOS_GSD, Q13 Q_NMOS_GSD, Q14 Q_NMOS_GSD, Q15 Q_NMOS_GSD, Q16 Q_NMOS_GSD, Q17 Q_NMOS_GSD, Q2 Q_NMOS_GSD, Q3 Q_NMOS_GSD, Q4 Q_NMOS_GSD, Q5 Q_NMOS_GSD, Q6 Q_NMOS_GSD, Q7 Q_NMOS_GSD, Q8 Q_NMOS_GSD, Q9 Q_NMOS_GSD, U1 DRV8833RTY, U10 74LVC2G14, U11 AP6503, U12 AP6503, U13 TXB0102DCU, U2 DRV8833RTY, U3 DRV8833RTY, U4 DRV8833RTY, U5 MCP3008, U6 CBT3245A, U7 CBT3245A, U8 INA4180, U9 INA4180

Commit message: Add capper v2 corrections
Parts:
- J4: footprint Connector_PinHeader_1.27mm:PinHeader_2x20_P1.27mm_Vertical -> Connector_PinSocket_2.54mm:PinSocket_2x20_P2.54mm_Vertical
Changed lines of the file:
@@
 Text Label 8150 8700 0    50   ~ 0
 SolSet
-Wire Wire Line
-	8500 8700 8150 8700
 NoConn ~ 8500 8500
 NoConn ~ 9000 9500
@@
 Wire Wire Line
 	9000 8500 9400 8500
-Wire Wire Line
-	8150 8800 8500 8800
 Text Label 8150 9000 0    50   ~ 0
 RunLedB
-Wire Wire Line
-	8150 8900 8500 8900
 Text Label 8150 8900 0    50   ~ 0
 RunLedR
-Wire Wire Line
-	8150 9000 8500 9000
 Text Label 8150 8800 0    50   ~ 0
 RunLedG
 Text Label 8300 8400 0    50   ~ 0
 SCL
-Wire Wire Line
-	8500 8400 8300 8400
-Wire Wire Line
-	8300 8300 8500 8300
 Text Label 8300 8300 0    50   ~ 0
 SDA
-Wire Wire Line
-	8500 9500 8200 9500
 Text Label 8200 9500 0    50   ~ 0
 Mot8En
-Wire Wire Line
-	8500 9600 8200 9600
 Text Label 8200 9600 0    50   ~ 0
 Mot7En
-Wire Wire Line
-	8500 9700 8200 9700
 Text Label 8200 9700 0    50   ~ 0
 Mot6En
-Wire Wire Line
-	8500 9900 8200 9900
 Text Label 8200 9900 0    50   ~ 0
 Mot5En
-Wire Wire Line
-	8500 10000 8200 10000
 Text Label 9300 10100 2    50   ~ 0
 Mot3En
@@
 Text Label 9300 9900 2    50   ~ 0
 Mot1En
-Wire Wire Line
-	8150 9800 8500 9800
 Text Label 8150 9800 0    50   ~ 0
 PwmFwd
@@
 Wire Wire Line
 	9000 9300 9250 9300
-Wire Wire Line
-	8250 9100 8500 9100
 Text Label 8250 9100 0    50   ~ 0
 MOSI
 Text Label 8250 9200 0    50   ~ 0
 MISO
-Wire Wire Line
-	8500 9200 8250 9200
 Text Label 8250 9300 0    50   ~ 0
 SCLK
-Wire Wire Line
-	8500 9300 8250 9300
 $Comp
 L power:GND #PWR056
@@
 	1    0    0    -1
 $EndComp
-Wire Wire Line
-	8500 9400 8100 9400
 $Comp
 L power:GND #PWR046
@@
 $EndComp
 Wire Wire Line
-	8500 8600 8000 8600
-Wire Wire Line
 	9000 8800 9500 8800
 Wire Wire Line
@@
 	1    0    0    -1
 $EndComp
-Wire Wire Line
-	8500 10100 8100 10100
 Wire Wire Line
 	9000 9800 9500 9800
@@
 	1    0    0    -1
 $EndComp
-Wire Wire Line
-	8500 8200 8300 8200
 Connection ~ 9150 8200
 $Comp
@@
 Wire Wire Line
 	9000 8200 9150 8200
-$Comp
-L Connector_Generic:Conn_02x20_Odd_Even J4
-U 1 1 5EE19EEA
-P 8700 9100
-F 0 "J4" H 8750 10150 50  0000 C CNN
-F 1 "Pi_Header" H 8800 8000 50  0000 C CNN
-F 2 "Connector_PinHeader_1.27mm:PinHeader_2x20_P1.27mm_Vertical" H 8700 9100 50  0001 C CNN
-F 3 "~" H 8700 9100 50  0001 C CNN
-	1    8700 9100
-	1    0    0    -1
-$EndComp
 Text Notes 9050 7950 2    79   ~ 16
 Pi Header
@@
 	1    0    0    -1
 $EndComp
+Wire Wire Line
+	8500 8400 8300 8400
+Wire Wire Line
+	8500 10100 8100 10100
+Wire Wire Line
+	8300 8300 8500 8300
+Wire Wire Line
+	8500 10000 8200 10000
+Wire Wire Line
+	8500 9900 8200 9900
+Wire Wire Line
+	8150 9800 8500 9800
+Wire Wire Line
+	8500 9700 8200 9700
+Wire Wire Line
+	8500 9600 8200 9600
+Wire Wire Line
+	8500 9500 8200 9500
+Wire Wire Line
+	8500 9400 8100 9400
+Wire Wire Line
+	8500 9300 8250 9300
+Wire Wire Line
+	8500 9200 8250 9200
+Wire Wire Line
+	8250 9100 8500 9100
+Wire Wire Line
+	8500 8200 8300 8200
+Wire Wire Line
+	8150 9000 8500 9000
+Wire Wire Line
+	8150 8900 8500 8900
+Wire Wire Line
+	8150 8800 8500 8800
+Wire Wire Line
+	8500 8700 8150 8700
+Wire Wire Line
+	8500 8600 8000 8600
+$Comp
+L Connector_Generic:Conn_02x20_Odd_Even J4
+U 1 1 5EE19EEA
+P 8700 9100
+F 0 "J4" H 8750 10150 50  0000 C CNN
+F 1 "Pi_Header" H 8800 8000 50  0000 C CNN
+F 2 "Connector_PinSocket_2.54mm:PinSocket_2x20_P2.54mm_Vertical" H 8700 9100 50  0001 C CNN
+F 3 "~" H 8700 9100 50  0001 C CNN
+	1    8700 9100
+	1    0    0    -1
+$EndComp
