File: designs/Vespucci/Display Module/D1_ILI6122_FT5446/D1_DisplayInterface.sch (KiCad schematic (older format))
At the start: 9 parts

Commit message: Update P1 Rev B, R1 Rev B, D1 Rev A
Parts:
- J?: footprint (none) -> Custom_Footprints:Amphenol_62674-08
- J?: footprint (none) -> Custom_Footprints:JUSHUO_AFC07-S40
- R?: value 2R -> 2R4
Connections:
- net labels added: +BATT, TP_SCL, TP_SDA, ~TP_INT, ~TP_RST
- net labels removed: SCL, SDA, VBUS
- wire segments 76 -> 78
Other:
- note added: "Design Notes\n1. Designed for YL050MG-3240\n2. ~INT~ requires input pullup\n3. LED driver 90% eff @ 60mA 12V to 24V\n4. TFT : 60mA max @ 3V3 (200mW)\n5. Backlight : 80mA max @ 20V 90% eff (1800mW) | 40mA typ @ 19V 90% eff (840mW)\n6. Touch Panel : 11mA typ @ 3V3 (36mW)"
- note added: "Output : 83mA Max"
- note added: "VIn : 12V"
Changed lines of the file:
@@
 $Descr A4 11693 8268
 encoding utf-8
-Sheet 2 6
+Sheet 4 7
 Title ""
 Date ""
@@
 AR Path="/5ECC709A" Ref="J?"  Part="1"
 AR Path="/5ECC290F/5ECC709A" Ref="J?"  Part="1"
+AR Path="/5EE97019/5ECC290F/5ECC709A" Ref="J?"  Part="1"
 F 0 "J?" H 9878 3176 50  0000 L CNN
 F 1 "FFC_FT5446" H 9878 3085 50  0000 L CNN
-F 2 "" H 9850 3200 50  0001 C CNN
-F 3 "~" H 9850 3200 50  0001 C CNN
+F 2 "Custom_Footprints:Amphenol_62674-08" H 9850 3200 50  0001 C CNN
+F 3 "https://cdn.amphenol-icc.com/media/wysiwyg/files/drawing/62674.pdf" H 9850 3200 50  0001 C CNN
 	1    9850 3200
 	1    0    0    -1
@@
 AR Path="/5ECC70A0" Ref="J?"  Part="1"
 AR Path="/5ECC290F/5ECC70A0" Ref="J?"  Part="1"
+AR Path="/5EE97019/5ECC290F/5ECC70A0" Ref="J?"  Part="1"
 F 0 "J?" H 6178 3976 50  0000 L CNN
 F 1 "FFC_ILI6122" H 6178 3885 50  0000 L CNN
-F 2 "" H 6150 4000 50  0001 C CNN
-F 3 "~" H 6150 4000 50  0001 C CNN
+F 2 "Custom_Footprints:JUSHUO_AFC07-S40" H 6150 4000 50  0001 C CNN
+F 3 "https://datasheet.lcsc.com/szlcsc/JUSHUO-AFC07-S40ECA-00_C262648.pdf" H 6150 4000 50  0001 C CNN
 	1    6150 4000
 	1    0    0    -1
@@
 AR Path="/5ECC7094" Ref="U?"  Part="1"
 AR Path="/5ECC290F/5ECC7094" Ref="U?"  Part="1"
+AR Path="/5EE97019/5ECC290F/5ECC7094" Ref="U?"  Part="1"
 F 0 "U?" H 2900 3200 50  0000 C CNN
 F 1 "TPS61165DRV" H 2900 2800 50  0000 C CNN
@@
 Wire Wire Line
 	5850 5400 5950 5400
-Text HLabel 5250 2400 0    50   BiDi ~ 0
+Text HLabel 5250 2400 0    50   Input ~ 0
 LCD_R[0..7]
 Entry Wire Line
@@
 Wire Bus Line
 	5350 2400 5250 2400
-Text HLabel 5250 3200 0    50   BiDi ~ 0
+Text HLabel 5250 3200 0    50   Input ~ 0
 LCD_G[0..7]
 Entry Wire Line
@@
 Wire Bus Line
 	5350 3200 5250 3200
-Text HLabel 5250 4000 0    50   BiDi ~ 0
+Text HLabel 5250 4000 0    50   Input ~ 0
 LCD_B[0..7]
 Entry Wire Line
@@
 P 3400 3450
 F 0 "R?" V 3500 3450 50  0000 C CNN
-F 1 "2R" V 3400 3450 50  0000 C CNN
+F 1 "2R4" V 3400 3450 50  0000 C CNN
 F 2 "" V 3330 3450 50  0001 C CNN
 F 3 "~" H 3400 3450 50  0001 C CNN
@@
 	3250 3450 3250 3350
 Connection ~ 3250 3350
-$Comp
-L power:VBUS #PWR?
-U 1 1 5FF08357
-P 2550 2600
-F 0 "#PWR?" H 2550 2450 50  0001 C CNN
-F 1 "VBUS" H 2565 2773 50  0000 C CNN
-F 2 "" H 2550 2600 50  0001 C CNN
-F 3 "" H 2550 2600 50  0001 C CNN
-	1    2550 2600
-	1    0    0    -1
-$EndComp
 Wire Wire Line
 	2550 2600 2550 2700
@@
 	9650 3000 9550 3000
 Wire Wire Line
-	9550 3000 9550 2950
-Wire Wire Line
 	9550 2900 9650 2900
 Wire Wire Line
 	9650 3500 9550 3500
 Wire Wire Line
-	9550 3500 9550 3550
-Wire Wire Line
 	9550 3600 9650 3600
 Wire Wire Line
-	9550 3550 9250 3550
-Wire Wire Line
-	9250 3550 9250 3500
-Connection ~ 9550 3550
-Wire Wire Line
-	9550 3550 9550 3600
+	9550 2950 9150 2950
+Wire Wire Line
+	9150 2950 9150 3000
+$Comp
+L power:GND #PWR?
+U 1 1 5FF71F03
+P 9150 3000
+F 0 "#PWR?" H 9150 2750 50  0001 C CNN
+F 1 "GND" H 9150 2850 50  0000 C CNN
+F 2 "" H 9150 3000 50  0001 C CNN
+F 3 "" H 9150 3000 50  0001 C CNN
+	1    9150 3000
+	1    0    0    -1
+$EndComp
+Wire Wire Line
+	9650 3400 9600 3400
+Wire Wire Line
+	9650 3300 9600 3300
+Wire Wire Line
+	9650 3200 9600 3200
+Text Notes 7000 7100 0    50   ~ 0
+Design Notes\n1. Designed for YL050MG-3240\n2. ~INT~ requires input pullup\n3. LED driver 90% eff @ 60mA 12V to 24V\n4. TFT : 60mA max @ 3V3 (200mW)\n5. Backlight : 80mA max @ 20V 90% eff (1800mW) | 40mA typ @ 19V 90% eff (840mW)\n6. Touch Panel : 11mA typ @ 3V3 (36mW)
 $Comp
 L power:+3V3 #PWR?
 U 1 1 5FF6FC1C
-P 9250 3500
-F 0 "#PWR?" H 9250 3350 50  0001 C CNN
-F 1 "+3V3" H 9265 3673 50  0000 C CNN
-F 2 "" H 9250 3500 50  0001 C CNN
-F 3 "" H 9250 3500 50  0001 C CNN
-	1    9250 3500
-	1    0    0    -1
-$EndComp
-Wire Wire Line
-	9550 2950 9250 2950
-Wire Wire Line
-	9250 2950 9250 3000
+P 9150 3500
+F 0 "#PWR?" H 9150 3350 50  0001 C CNN
+F 1 "+3V3" H 9100 3650 50  0000 C CNN
+F 2 "" H 9150 3500 50  0001 C CNN
+F 3 "" H 9150 3500 50  0001 C CNN
+	1    9150 3500
+	1    0    0    -1
+$EndComp
+Wire Wire Line
+	9150 3550 9150 3500
+Text HLabel 9600 3100 0    50   Input ~ 0
+~TP_RST
+Wire Wire Line
+	9600 3100 9650 3100
+Text HLabel 9600 3200 0    50   Output ~ 0
+~TP_INT
+Wire Wire Line
+	9550 2900 9550 2950
 Connection ~ 9550 2950
 Wire Wire Line
-	9550 2950 9550 2900
-$Comp
-L power:GND #PWR?
-U 1 1 5FF71F03
-P 9250 3000
-F 0 "#PWR?" H 9250 2750 50  0001 C CNN
-F 1 "GND" H 9255 2827 50  0000 C CNN
-F 2 "" H 9250 3000 50  0001 C CNN
-F 3 "" H 9250 3000 50  0001 C CNN
-	1    9250 3000
-	1    0    0    -1
-$EndComp
-Wire Wire Line
-	9650 3400 9450 3400
-Text Label 9450 3400 0    50   ~ 0
-SCL
-Wire Wire Line
-	9650 3300 9450 3300
+	9550 2950 9550 3000
+Wire Wire Line
+	9550 3500 9550 3550
+Wire Wire Line
+	9150 3550 9550 3550
+Connection ~ 9550 3550
+Wire Wire Line
+	9550 3550 9550 3600
+Text HLabel 9600 3300 0    50   BiDi ~ 0
+TP_SDA
+Text HLabel 9600 3400 0    50   Input ~ 0
+TP_SCL
 Wire Bus Line
 	5350 2400 5350 3100
@@
 Wire Bus Line
 	5350 4000 5350 4700
-Text Label 9450 3300 0    50   ~ 0
-SDA
+$Comp
+L power:+BATT #PWR?
+U 1 1 5F7D6978
+P 2550 2600
+F 0 "#PWR?" H 2550 2450 50  0001 C CNN
+F 1 "+BATT" H 2565 2773 50  0000 C CNN
+F 2 "" H 2550 2600 50  0001 C CNN
+F 3 "" H 2550 2600 50  0001 C CNN
+	1    2550 2600
+	1    0    0    -1
+$EndComp
+Text Notes 2250 2200 0    79   ~ 16
+VIn : 12V
+Text Notes 3000 2200 0    79   ~ 16
+Output : 83mA Max
 $EndSCHEMATC

Commit message: R4R D1 Rev A
Parts:
- C1, C2, C3: renamed from C?; footprint (none) -> Capacitor_SMD:C_0402_1005Metric
- J2: renamed from J?; footprint Custom_Footprints:JUSHUO_AFC07-S40 -> Custom_Footprints:JUSHUO_AFC11_S40IC
- R12: renamed from R?; footprint (none) -> Resistor_SMD:R_0402_1005Metric
- gave numbers to parts that had none: 4
Connections:
- net labels removed: LCD_B0
Changed lines of the file:
@@
 $Descr A4 11693 8268
 encoding utf-8
-Sheet 4 7
+Sheet 2 4
 Title ""
 Date ""
@@
 P 9850 3200
 AR Path="/5ECC709A" Ref="J?"  Part="1"
-AR Path="/5ECC290F/5ECC709A" Ref="J?"  Part="1"
+AR Path="/5ECC290F/5ECC709A" Ref="J3"  Part="1"
 AR Path="/5EE97019/5ECC290F/5ECC709A" Ref="J?"  Part="1"
-F 0 "J?" H 9878 3176 50  0000 L CNN
+F 0 "J3" H 9878 3176 50  0000 L CNN
 F 1 "FFC_FT5446" H 9878 3085 50  0000 L CNN
 F 2 "Custom_Footprints:Amphenol_62674-08" H 9850 3200 50  0001 C CNN
@@
 P 6150 4000
 AR Path="/5ECC70A0" Ref="J?"  Part="1"
-AR Path="/5ECC290F/5ECC70A0" Ref="J?"  Part="1"
+AR Path="/5ECC290F/5ECC70A0" Ref="J2"  Part="1"
 AR Path="/5EE97019/5ECC290F/5ECC70A0" Ref="J?"  Part="1"
-F 0 "J?" H 6178 3976 50  0000 L CNN
+F 0 "J2" H 6178 3976 50  0000 L CNN
 F 1 "FFC_ILI6122" H 6178 3885 50  0000 L CNN
-F 2 "Custom_Footprints:JUSHUO_AFC07-S40" H 6150 4000 50  0001 C CNN
+F 2 "Custom_Footprints:JUSHUO_AFC11_S40IC" H 6150 4000 50  0001 C CNN
 F 3 "https://datasheet.lcsc.com/szlcsc/JUSHUO-AFC07-S40ECA-00_C262648.pdf" H 6150 4000 50  0001 C CNN
 	1    6150 4000
@@
 P 2900 3000
 AR Path="/5ECC7094" Ref="U?"  Part="1"
-AR Path="/5ECC290F/5ECC7094" Ref="U?"  Part="1"
+AR Path="/5ECC290F/5ECC7094" Ref="U3"  Part="1"
 AR Path="/5EE97019/5ECC290F/5ECC7094" Ref="U?"  Part="1"
-F 0 "U?" H 2900 3200 50  0000 C CNN
+F 0 "U3" H 2900 3200 50  0000 C CNN
 F 1 "TPS61165DRV" H 2900 2800 50  0000 C CNN
 F 2 "Package_SON:WSON-6-1EP_2x2mm_P0.65mm_EP1x1.6mm_ThermalVias" H 2450 3300 50  0001 C CNN
@@
 Text HLabel 5250 4000 0    50   Input ~ 0
 LCD_B[0..7]
-Entry Wire Line
-	5450 4100 5350 4000
 Text Label 5850 4800 2    50   ~ 0
 LCD_B7
@@
 Text Label 5850 4200 2    50   ~ 0
 LCD_B1
-Text Label 5850 4100 2    50   ~ 0
-LCD_B0
 Entry Wire Line
 	5450 4800 5350 4700
@@
 Entry Wire Line
 	5450 4200 5350 4100
-Wire Wire Line
-	5450 4100 5950 4100
 Wire Wire Line
 	5450 4200 5950 4200
@@
 	5950 2300 5650 2300
 $Comp
-L power:+3V3 #PWR?
+L power:+3V3 #PWR022
 U 1 1 5FE7D658
 P 5450 2150
-F 0 "#PWR?" H 5450 2000 50  0001 C CNN
+F 0 "#PWR022" H 5450 2000 50  0001 C CNN
 F 1 "+3V3" H 5300 2200 50  0000 C CNN
 F 2 "" H 5450 2150 50  0001 C CNN
@@
 	5350 4900 5350 5600
 $Comp
-L power:GND #PWR?
+L power:GND #PWR021
 U 1 1 5FE88588
 P 5350 5650
-F 0 "#PWR?" H 5350 5400 50  0001 C CNN
+F 0 "#PWR021" H 5350 5400 50  0001 C CNN
 F 1 "GND" H 5355 5477 50  0000 C CNN
 F 2 "" H 5350 5650 50  0001 C CNN
@@
 	3250 2700 3250 2900
 $Comp
-L Device:D D?
+L Device:D D7
 U 1 1 5FEEB906
 P 3500 2700
-F 0 "D?" H 3500 2483 50  0000 C CNN
+F 0 "D7" H 3500 2483 50  0000 C CNN
 F 1 "MBR0540" H 3500 2574 50  0000 C CNN
 F 2 "Diode_SMD:D_SOD-123" H 3500 2700 50  0001 C CNN
@@
 	3750 2700 3750 3000
 $Comp
-L Device:C C?
+L Device:C C3
 U 1 1 5FEEE945
 P 3750 3150
-F 0 "C?" H 3800 3350 50  0000 L CNN
+F 0 "C3" H 3800 3350 50  0000 L CNN
 F 1 "4.7uF" H 3800 3250 50  0000 L CNN
-F 2 "" H 3788 3000 50  0001 C CNN
+F 2 "Capacitor_SMD:C_0402_1005Metric" H 3788 3000 50  0001 C CNN
 F 3 "~" H 3750 3150 50  0001 C CNN
 	1    3750 3150
@@
 LED+
 $Comp
-L Device:C C?
+L Device:C C2
 U 1 1 5FEF1F64
 P 3450 3150
-F 0 "C?" H 3500 3350 50  0000 L CNN
+F 0 "C2" H 3500 3350 50  0000 L CNN
 F 1 "220nF" H 3450 3250 50  0000 L CNN
-F 2 "" H 3488 3000 50  0001 C CNN
+F 2 "Capacitor_SMD:C_0402_1005Metric" H 3488 3000 50  0001 C CNN
 F 3 "~" H 3450 3150 50  0001 C CNN
 	1    3450 3150
@@
 	3600 3300 3750 3300
 $Comp
-L power:GND #PWR?
+L power:GND #PWR020
 U 1 1 5FEF9E84
 P 3600 3550
-F 0 "#PWR?" H 3600 3300 50  0001 C CNN
+F 0 "#PWR020" H 3600 3300 50  0001 C CNN
 F 1 "GND" H 3605 3377 50  0000 C CNN
 F 2 "" H 3600 3550 50  0001 C CNN
@@
 	2550 3100 2550 3200
 $Comp
-L power:GND #PWR?
+L power:GND #PWR019
 U 1 1 5FEFBB78
 P 2550 3200
-F 0 "#PWR?" H 2550 2950 50  0001 C CNN
+F 0 "#PWR019" H 2550 2950 50  0001 C CNN
 F 1 "GND" H 2555 3027 50  0000 C CNN
 F 2 "" H 2550 3200 50  0001 C CNN
@@
 LED-
 $Comp
-L Device:R R?
+L Device:R R12
 U 1 1 5FF00AB4
 P 3400 3450
-F 0 "R?" V 3500 3450 50  0000 C CNN
+F 0 "R12" V 3500 3450 50  0000 C CNN
 F 1 "2R4" V 3400 3450 50  0000 C CNN
-F 2 "" V 3330 3450 50  0001 C CNN
+F 2 "Resistor_SMD:R_0402_1005Metric" V 3330 3450 50  0001 C CNN
 F 3 "~" H 3400 3450 50  0001 C CNN
 	1    3400 3450
@@
 Connection ~ 2550 2700
 $Comp
-L Device:C C?
+L Device:C C1
 U 1 1 5FF0AA7D
 P 2400 2700
-F 0 "C?" V 2550 2800 50  0000 L CNN
+F 0 "C1" V 2550 2800 50  0000 L CNN
 F 1 "4.7uF" V 2450 2750 50  0000 L CNN
-F 2 "" H 2438 2550 50  0001 C CNN
+F 2 "Capacitor_SMD:C_0402_1005Metric" H 2438 2550 50  0001 C CNN
 F 3 "~" H 2400 2700 50  0001 C CNN
 	1    2400 2700
@@
 	2250 2700 2150 2700
 $Comp
-L power:GND #PWR?
+L power:GND #PWR017
 U 1 1 5FF0DBBD
 P 2150 2700
-F 0 "#PWR?" H 2150 2450 50  0001 C CNN
+F 0 "#PWR017" H 2150 2450 50  0001 C CNN
 F 1 "GND" H 2155 2527 50  0000 C CNN
 F 2 "" H 2150 2700 50  0001 C CNN
@@
 LCD_PWM
 $Comp
-L Device:L L?
+L Device:L L1
 U 1 1 5FEE62DB
 P 2900 2700
-F 0 "L?" V 3090 2700 50  0000 C CNN
+F 0 "L1" V 3090 2700 50  0000 C CNN
 F 1 "10uH" V 2999 2700 50  0000 C CNN
 F 2 "Inductor_SMD:L_1210_3225Metric" H 2900 2700 50  0001 C CNN
@@
 	5650 2050 5550 2050
 $Comp
-L power:GND #PWR?
+L power:GND #PWR023
 U 1 1 5FF20216
 P 5550 2100
-F 0 "#PWR?" H 5550 1850 50  0001 C CNN
+F 0 "#PWR023" H 5550 1850 50  0001 C CNN
 F 1 "GND" H 5555 1927 50  0000 C CNN
 F 2 "" H 5550 2100 50  0001 C CNN
@@
 	9150 2950 9150 3000
 $Comp
-L power:GND #PWR?
+L power:GND #PWR024
 U 1 1 5FF71F03
 P 9150 3000
-F 0 "#PWR?" H 9150 2750 50  0001 C CNN
+F 0 "#PWR024" H 9150 2750 50  0001 C CNN
 F 1 "GND" H 9150 2850 50  0000 C CNN
 F 2 "" H 9150 3000 50  0001 C CNN
@@
 Design Notes\n1. Designed for YL050MG-3240\n2. ~INT~ requires input pullup\n3. LED driver 90% eff @ 60mA 12V to 24V\n4. TFT : 60mA max @ 3V3 (200mW)\n5. Backlight : 80mA max @ 20V 90% eff (1800mW) | 40mA typ @ 19V 90% eff (840mW)\n6. Touch Panel : 11mA typ @ 3V3 (36mW)
 $Comp
-L power:+3V3 #PWR?
+L power:+3V3 #PWR025
 U 1 1 5FF6FC1C
 P 9150 3500
-F 0 "#PWR?" H 9150 3350 50  0001 C CNN
+F 0 "#PWR025" H 9150 3350 50  0001 C CNN
 F 1 "+3V3" H 9100 3650 50  0000 C CNN
 F 2 "" H 9150 3500 50  0001 C CNN
@@
 Text HLabel 9600 3400 0    50   Input ~ 0
 TP_SCL
+$Comp
+L power:+BATT #PWR018
+U 1 1 5F7D6978
+P 2550 2600
+F 0 "#PWR018" H 2550 2450 50  0001 C CNN
+F 1 "+BATT" H 2565 2773 50  0000 C CNN
+F 2 "" H 2550 2600 50  0001 C CNN
+F 3 "" H 2550 2600 50  0001 C CNN
+	1    2550 2600
+	1    0    0    -1
+$EndComp
+Text Notes 2250 2200 0    79   ~ 16
+VIn : 12V
+Text Notes 3000 2200 0    79   ~ 16
+Output : 83mA Max
+$Comp
+L custom-components:OSHW_logo #G1
+U 1 1 5F279257
+P 11100 7250
+F 0 "#G1" H 11100 7180 60  0001 C CNN
+F 1 "OSHW_logo" H 11100 7320 60  0001 C CNN
+F 2 "Custom_Footprints:OSHW_logo" H 11100 7250 50  0001 C CNN
+F 3 "" H 11100 7250 50  0001 C CNN
+	1    11100 7250
+	1    0    0    -1
+$EndComp
+Wire Wire Line
+	5950 4100 5700 4100
+Text Label 5700 4100 0    50   ~ 0
+GND
 Wire Bus Line
 	5350 2400 5350 3100
@@
 Wire Bus Line
 	5350 4000 5350 4700
-$Comp
-L power:+BATT #PWR?
-U 1 1 5F7D6978
-P 2550 2600
-F 0 "#PWR?" H 2550 2450 50  0001 C CNN
-F 1 "+BATT" H 2565 2773 50  0000 C CNN
-F 2 "" H 2550 2600 50  0001 C CNN
-F 3 "" H 2550 2600 50  0001 C CNN
-	1    2550 2600
-	1    0    0    -1
-$EndComp
-Text Notes 2250 2200 0    79   ~ 16
-VIn : 12V
-Text Notes 3000 2200 0    79   ~ 16
-Output : 83mA Max
 $EndSCHEMATC

Commit message: Ordered: D1 Rev A, R1 Rev B, P1 Rev B
Other:
- note added: "1. Designed for YL050MG-3240\n2. ~INT~ requires input pullup\n3. LED driver 90% eff @ 60mA 12V to 24V\n4. TFT : 60mA max @ 3V3 (200mW)\n5. Backlight : 80mA max @ 20V 90% eff (1800mW) | 40mA typ @ 19V 90% eff (840mW)\n6. Touch Panel : 11mA typ @ 3V3 (36mW)"
- note added: "LCD Backlight Current Driver"
- note added: "LCD Connector"
- note added: "Touch Panel Connector"
- note removed: "Design Notes\n1. Designed for YL050MG-3240\n2. ~INT~ requires input pullup\n3. LED driver 90% eff @ 60mA 12V to 24V\n4. TFT : 60mA max @ 3V3 (200mW)\n5. Backlight : 80mA max @ 20V 90% eff (1800mW) | 40mA typ @ 19V 90% eff (840mW)\n6. Touch Panel : 11mA typ @ 3V3 (36mW)"

Commit message: M1 Rev A, minor component changes in schematic
Parts:
- D7: value MBR0540 -> LMBR3100FT1G; footprint Diode_SMD:D_SOD-123 -> Diode_SMD:D_SOD-123F
Changed lines of the file:
@@
 P 3150 2650
 F 0 "D7" H 3150 2433 50  0000 C CNN
-F 1 "MBR0540" H 3150 2524 50  0000 C CNN
-F 2 "Diode_SMD:D_SOD-123" H 3150 2650 50  0001 C CNN
+F 1 "LMBR3100FT1G" H 3150 2524 50  0000 C CNN
+F 2 "Diode_SMD:D_SOD-123F" H 3150 2650 50  0001 C CNN
 F 3 "https://datasheet.lcsc.com/szlcsc/1809181018_ON-Semiconductor-MBR0540_C232833.pdf" H 3150 2650 50  0001 C CNN
 	1    3150 2650
