File: designs/Vespucci/Display Module/D1_ILI6122_FT5446/D1_ILI6122_FT5446.sch (KiCad schematic (older format))
At the start: 0 parts

Commit message: Update P1 Rev B, R1 Rev B, D1 Rev A
Parts:
- added D? (x3): LED, LED_SMD:LED_0603_1608Metric, symbol Device:LED
- added H? (x2): MountingHole_Pad, MountingHole:MountingHole_2.7mm_M2.5_ISO7380_Pad, symbol Mechanical:MountingHole_Pad
- added J?: PCIExpress, Connector_PCBEdge:BUS_PCIexpress_x1, symbol Connector_Generic:Conn_02x18_Row_Letter_First
- added Q? (x2): BSS138W, Package_TO_SOT_SMD:SOT-323_SC-70, symbol Device:Q_NMOS_GSD
- added R? (x3): 470R, Resistor_SMD:R_0402_1005Metric, symbol Device:R
- added R?: 1K2, symbol Device:R
- added R?: 8K41, symbol Device:R
- added R?: 51K, Resistor_SMD:R_0402_1005Metric, symbol Device:R
- added R?: 51K, symbol Device:R
- added U? (x2): NC7WZ14, Package_TO_SOT_SMD:SOT-363_SC-70-6, symbol custom-components:NC7WZ14
Connections:
- net labels added: +BATT, GND, LED_RX, LED_TX, PRSNT, PWROK, SMCLK, SMDAT, SW_PWR, SYSID, TCK, TDI, TDO, TMS, VBUS, VDD_EXT, hCTS, hDCD, hDTR, hRI, hRTS, hRX, hTX, ~TRST
- wire segments 5 -> 134
- no-connect marks 0 -> 2
Other:
- note added: "Design Notes:\n1. Total max current consumption - 3V3: 386mA; 12V: 150mA\n2. Total max power consumption - 3000mW"
- note added: "Interfaces"
- note added: "PCIe"
- note added: "SYSID : 0.875"
- note added: "VBatt : 12V"
- note added: "VBus : 3V3"
- note removed: "Design Notes\n1. LCD clock is PLLSAI\n2. USART1/6 have 11.25Mbit/s\n3. SPI1/4/5/6 have 45Mbit/s\n4. Temperature sensor is ADC1_IN18\n5. JTAG and SWD share the same pins. TMS switches modes\n6.PA13-JTMS//PA14-JTCK//PA15-JTDI//PB3-JTDO//PB4-NJTRST"

Commit message: R4R D1 Rev A
Parts:
- removed Q?: BSS138W, Package_TO_SOT_SMD:SOT-323_SC-70, symbol Device:Q_NMOS_GSD
- removed R?: 51K, symbol Device:R
- added D4, D5, D6: LED, LED_SMD:LED_0603_1608Metric, symbol Device:LED
- added G1: OSHW_logo, Custom_Footprints:OSHW_logo, symbol custom-components:OSHW_logo
- added Q3: BSS138W, Package_TO_SOT_SMD:SOT-323_SC-70, symbol Device:Q_NMOS_GSD
- added R6: 51K, Resistor_SMD:R_0402_1005Metric, symbol Device:R
- added R7, R8, R9: 470R, Resistor_SMD:R_0402_1005Metric, symbol Device:R
- added U2: NC7WZ14, Package_TO_SOT_SMD:SOT-363_SC-70-6, symbol custom-components:NC7WZ14
- R10, R11: renamed from R?; footprint (none) -> Resistor_SMD:R_0402_1005Metric
- gave numbers to parts that had none: 12
Connections:
- net labels added: +3V3, LCD_ON, ~SLEEP, ~TP_INT
- net labels removed: LED_RX, LED_TX, SW_PWR, VDD_EXT
- wire segments 134 -> 144
Other:
- note added: "PCIe Interface"
- note removed: "Interfaces"
- note removed: "PCIe"

Commit message: Ordered: D1 Rev A, R1 Rev B, P1 Rev B
Other:
- note added: "Interconnects"
- note added: "LCD and Touch Panel"
- note added: "LEDs"
- note added: "Misc."
- note added: "NOR Flash"
- note added: "STM32F429"
