File: designs/Vespucci/Display Module/D1_ILI6122_FT5446/D1_SST39VF3201C.sch (KiCad schematic (older format))
At the start: 4 parts

Commit message: Update P1 Rev B, R1 Rev B, D1 Rev A
Parts:
- C?: value 100nF -> 1uF
Other:
- note added: "Design Notes:\n1. NOR Flash : 45mA max @ 3V3 (150mW)"
Changed lines of the file:
@@
 $Descr A4 11693 8268
 encoding utf-8
-Sheet 4 6
+Sheet 5 7
 Title ""
 Date ""
@@
 P 5950 2100
 F 0 "C?" V 5698 2100 50  0000 C CNN
-F 1 "100nF" V 5789 2100 50  0000 C CNN
+F 1 "1uF" V 5789 2100 50  0000 C CNN
 F 2 "" H 5988 1950 50  0001 C CNN
 F 3 "~" H 5950 2100 50  0001 C CNN
@@
 Text HLabel 6850 4800 2    50   Output ~ 0
 NOR_nWAIT
+Text Notes 7000 6700 0    50   ~ 0
+Design Notes:\n1. NOR Flash : 45mA max @ 3V3 (150mW)
 Wire Bus Line
 	6600 2300 6600 3900

Commit message: R4R D1 Rev A
Parts:
- C4: renamed from C?; footprint (none) -> Capacitor_SMD:C_0402_1005Metric
- R13, R14: renamed from R?; footprint (none) -> Resistor_SMD:R_0402_1005Metric
- gave numbers to parts that had none: 1
Connections:
- net labels added: A[0..20]
- net labels removed: A[0..15]
Changed lines of the file:
@@
 $Descr A4 11693 8268
 encoding utf-8
-Sheet 5 7
+Sheet 3 4
 Title ""
 Date ""
@@
 U 1 1 5ECB6EA6
 P 5700 3650
-F 0 "U?" H 4900 2550 50  0000 C CNN
+AR Path="/5ECB6EA6" Ref="U?"  Part="1"
+AR Path="/5ECA9B33/5ECB6EA6" Ref="U4"  Part="1"
+AR Path="/5ECC7549/5ECB6EA6" Ref="U4"  Part="1"
+F 0 "U4" H 4900 2550 50  0000 C CNN
 F 1 "SST39VF3201C-70-4I-B3KE" H 5000 2400 50  0000 C CNN
 F 2 "Custom_Footprints:TFBGA-48_6x8_6.0x8.0mm" H 5700 3950 50  0001 C CNN
@@
 	6300 4200 7000 4200
 $Comp
-L Device:R R?
+L Device:R R13
 U 1 1 5ECB6F20
 P 7150 4200
-F 0 "R?" V 7050 4200 50  0000 C CNN
+F 0 "R13" V 7050 4200 50  0000 C CNN
 F 1 "39K" V 7150 4200 50  0000 C CNN
-F 2 "" V 7080 4200 50  0001 C CNN
+F 2 "Resistor_SMD:R_0402_1005Metric" V 7080 4200 50  0001 C CNN
 F 3 "~" H 7150 4200 50  0001 C CNN
 	1    7150 4200
@@
 	5700 5100 5750 5100
 $Comp
-L power:GND #PWR?
+L power:GND #PWR027
 U 1 1 5ECB6F2C
 P 5700 5200
-F 0 "#PWR?" H 5700 4950 50  0001 C CNN
+F 0 "#PWR027" H 5700 4950 50  0001 C CNN
 F 1 "GND" H 5705 5027 50  0000 C CNN
 F 2 "" H 5700 5200 50  0001 C CNN
@@
 	6300 4500 6400 4500
 $Comp
-L power:+3V3 #PWR?
+L power:+3V3 #PWR026
 U 1 1 5ECB6F34
 P 5700 2000
-F 0 "#PWR?" H 5700 1850 50  0001 C CNN
+F 0 "#PWR026" H 5700 1850 50  0001 C CNN
 F 1 "+3V3" H 5715 2173 50  0000 C CNN
 F 2 "" H 5700 2000 50  0001 C CNN
@@
 	7300 4200 7300 4100
 $Comp
-L power:+3V3 #PWR?
+L power:+3V3 #PWR029
 U 1 1 5ECB6F3B
 P 7300 4100
-F 0 "#PWR?" H 7300 3950 50  0001 C CNN
+F 0 "#PWR029" H 7300 3950 50  0001 C CNN
 F 1 "+3V3" H 7315 4273 50  0000 C CNN
 F 2 "" H 7300 4100 50  0001 C CNN
@@
 $EndComp
 $Comp
-L Device:R R?
+L Device:R R14
 U 1 1 5ECB6F41
 P 7150 4600
-F 0 "R?" V 7050 4600 50  0000 C CNN
+F 0 "R14" V 7050 4600 50  0000 C CNN
 F 1 "39K" V 7150 4600 50  0000 C CNN
-F 2 "" V 7080 4600 50  0001 C CNN
+F 2 "Resistor_SMD:R_0402_1005Metric" V 7080 4600 50  0001 C CNN
 F 3 "~" H 7150 4600 50  0001 C CNN
 	1    7150 4600
@@
 	5700 2200 5700 2100
 $Comp
-L Device:C C?
+L Device:C C4
 U 1 1 5ECB6F56
 P 5950 2100
-F 0 "C?" V 5698 2100 50  0000 C CNN
+F 0 "C4" V 5698 2100 50  0000 C CNN
 F 1 "1uF" V 5789 2100 50  0000 C CNN
-F 2 "" H 5988 1950 50  0001 C CNN
+F 2 "Capacitor_SMD:C_0402_1005Metric" H 5988 1950 50  0001 C CNN
 F 3 "~" H 5950 2100 50  0001 C CNN
 	1    5950 2100
@@
 	6100 2100 6200 2100
 $Comp
-L power:GND #PWR?
+L power:GND #PWR028
 U 1 1 5ECB6F60
 P 6200 2100
-F 0 "#PWR?" H 6200 1850 50  0001 C CNN
+F 0 "#PWR028" H 6200 1850 50  0001 C CNN
 F 1 "GND" H 6205 1927 50  0000 C CNN
 F 2 "" H 6200 2100 50  0001 C CNN
@@
 D[0..15]
 Text HLabel 4700 2300 0    50   Input ~ 0
-A[0..15]
+A[0..20]
 Text HLabel 6400 4300 2    50   Input ~ 0
 NOR_RST
@@
 Text Notes 7000 6700 0    50   ~ 0
 Design Notes:\n1. NOR Flash : 45mA max @ 3V3 (150mW)
+$Comp
+L custom-components:OSHW_logo #G2
+U 1 1 5F27C4E9
+P 11100 7250
+F 0 "#G2" H 11100 7180 60  0001 C CNN
+F 1 "OSHW_logo" H 11100 7320 60  0001 C CNN
+F 2 "Custom_Footprints:OSHW_logo" H 11100 7250 50  0001 C CNN
+F 3 "" H 11100 7250 50  0001 C CNN
+	1    11100 7250
+	1    0    0    -1
+$EndComp
 Wire Bus Line
 	6600 2300 6600 3900

Commit message: Ordered: D1 Rev A, R1 Rev B, P1 Rev B
Parts:
- renumbered R14 to R13, R13 to R3
Changed lines of the file:
@@
 $Descr A4 11693 8268
 encoding utf-8
-Sheet 3 4
-Title ""
+Sheet 4 4
+Title "D1 NOR Flash"
 Date ""
 Rev ""
-Comp ""
+Comp "Puccinelli Laboratories, Inc"
 Comment1 ""
 Comment2 ""
@@
 	6300 4200 7000 4200
 $Comp
-L Device:R R13
+L Device:R R3
 U 1 1 5ECB6F20
 P 7150 4200
-F 0 "R13" V 7050 4200 50  0000 C CNN
+F 0 "R3" V 7050 4200 50  0000 C CNN
 F 1 "39K" V 7150 4200 50  0000 C CNN
 F 2 "Resistor_SMD:R_0402_1005Metric" V 7080 4200 50  0001 C CNN
@@
 	5700 5100 5750 5100
 $Comp
-L power:GND #PWR027
+L power:GND #PWR0103
 U 1 1 5ECB6F2C
 P 5700 5200
-F 0 "#PWR027" H 5700 4950 50  0001 C CNN
+F 0 "#PWR0103" H 5700 4950 50  0001 C CNN
 F 1 "GND" H 5705 5027 50  0000 C CNN
 F 2 "" H 5700 5200 50  0001 C CNN
@@
 	6300 4500 6400 4500
 $Comp
-L power:+3V3 #PWR026
+L power:+3V3 #PWR0104
 U 1 1 5ECB6F34
 P 5700 2000
-F 0 "#PWR026" H 5700 1850 50  0001 C CNN
+F 0 "#PWR0104" H 5700 1850 50  0001 C CNN
 F 1 "+3V3" H 5715 2173 50  0000 C CNN
 F 2 "" H 5700 2000 50  0001 C CNN
@@
 	7300 4200 7300 4100
 $Comp
-L power:+3V3 #PWR029
+L power:+3V3 #PWR0105
 U 1 1 5ECB6F3B
 P 7300 4100
-F 0 "#PWR029" H 7300 3950 50  0001 C CNN
+F 0 "#PWR0105" H 7300 3950 50  0001 C CNN
 F 1 "+3V3" H 7315 4273 50  0000 C CNN
 F 2 "" H 7300 4100 50  0001 C CNN
@@
 $EndComp
 $Comp
-L Device:R R14
+L Device:R R13
 U 1 1 5ECB6F41
 P 7150 4600
-F 0 "R14" V 7050 4600 50  0000 C CNN
+F 0 "R13" V 7050 4600 50  0000 C CNN
 F 1 "39K" V 7150 4600 50  0000 C CNN
 F 2 "Resistor_SMD:R_0402_1005Metric" V 7080 4600 50  0001 C CNN
@@
 	6100 2100 6200 2100
 $Comp
-L power:GND #PWR028
+L power:GND #PWR0106
 U 1 1 5ECB6F60
 P 6200 2100
-F 0 "#PWR028" H 6200 1850 50  0001 C CNN
+F 0 "#PWR0106" H 6200 1850 50  0001 C CNN
 F 1 "GND" H 6205 1927 50  0000 C CNN
 F 2 "" H 6200 2100 50  0001 C CNN
