File: designs/Vespucci/Display Module/D1_ILI6122_FT5446/D1_STM32F429.sch (KiCad schematic (older format))
At the start: 24 parts

Commit message: Update P1 Rev B, R1 Rev B, D1 Rev A
Connections:
- net labels added: I2C1_SCL, I2C1_SDA, I2C_SCL, I2C_SDA, USART_DCD, USART_DSR, USART_RI, ~JTRST, ~TP_INT, ~TP_RST
- net labels removed: USART1_CK, USART_CK, nJTRST
- wire segments 323 -> 334
Other:
- note added: "Design Notes\n1. USART1/6 supports 11.25Mbit/s max\n2. All I2C support 100kHz and 400kHz modes\n3. Temperature sensor is ADC1_IN18\n4. STM32F429 : 270mA max @ 3V3 (900mW)"
Changed lines of the file:
@@
 $Descr A4 11693 8268
 encoding utf-8
-Sheet 4 6
+Sheet 6 7
 Title ""
 Date ""
@@
 AR Path="/5ECDEA39" Ref="U?"  Part="1"
 AR Path="/5ECC7549/5ECDEA39" Ref="U?"  Part="1"
+AR Path="/5EE97019/5ECC7549/5ECDEA39" Ref="U?"  Part="1"
 F 0 "U?" V 4100 5850 50  0000 R CNN
 F 1 "STM32F429IGTx" V 5500 3450 50  0000 R CNN
@@
 Text Label 9000 4950 1    50   ~ 0
 LCD_G2
-Text Label 7900 4950 1    50   ~ 0
+Text Label 5300 1250 3    50   ~ 0
 LCD_R3
 Text Label 7800 4950 1    50   ~ 0
@@
 LCD_G6
 Text Label 8800 4950 1    50   ~ 0
-USART1_CK
+USART_DSR
 Text Label 8700 4950 1    50   ~ 0
 USART1_TX
@@
 JTDO
 Text Label 7500 4950 1    50   ~ 0
-nJTRST
+~JTRST
 Text Label 7100 4950 1    50   ~ 0
 LCD_B6
@@
 	9000 4550 9000 4950
 Wire Wire Line
-	7900 4550 7900 4950
+	5300 1650 5300 1250
 Wire Wire Line
 	7800 4550 7800 4950
@@
 RST
 Wire Wire Line
-	8600 5550 8600 5450
-Connection ~ 8600 5550
-$Comp
-L power:+3V3 #PWR?
-U 1 1 5F6736B0
-P 8600 5450
-F 0 "#PWR?" H 8600 5300 50  0001 C CNN
-F 1 "+3V3" H 8615 5623 50  0000 C CNN
-F 2 "" H 8600 5450 50  0001 C CNN
-F 3 "" H 8600 5450 50  0001 C CNN
-	1    8600 5450
-	1    0    0    -1
-$EndComp
-Wire Wire Line
 	7100 1650 7100 1300
 Entry Wire Line
@@
 Entry Wire Line
 	3850 6150 3950 6250
-Text HLabel 3650 6150 0    50   BiDi ~ 0
+Text HLabel 3650 6150 0    50   Output ~ 0
 LCD_R[0..7]
 Entry Wire Line
@@
 Entry Wire Line
 	3850 6700 3950 6800
-Text HLabel 3650 6700 0    50   BiDi ~ 0
+Text HLabel 3650 6700 0    50   Output ~ 0
 LCD_G[0..7]
 Entry Wire Line
@@
 Entry Wire Line
 	3850 7250 3950 7350
-Text HLabel 3650 7250 0    50   BiDi ~ 0
+Text HLabel 3650 7250 0    50   Output ~ 0
 LCD_B[0..7]
 Text Label 4100 5800 2    50   ~ 0
@@
 Wire Wire Line
 	8950 1000 9000 1000
-Text Label 6100 6800 2    50   ~ 0
+Text Label 6200 6600 2    50   ~ 0
 JTMS
 Wire Wire Line
-	5600 6800 6100 6800
-Text HLabel 5600 6800 0    50   Input ~ 0
+	5700 6600 6200 6600
+Text HLabel 5700 6600 0    50   Input ~ 0
 JTMS
-Text HLabel 5600 6700 0    50   Input ~ 0
-nJTRST
-Text HLabel 5600 7000 0    50   Input ~ 0
+Text HLabel 5700 6500 0    50   Input ~ 0
+~JTRST
+Text HLabel 5700 6800 0    50   Input ~ 0
 JTDI
 Wire Wire Line
-	5600 6700 6100 6700
-Wire Wire Line
-	5600 7000 6100 7000
-Text Label 6100 6700 2    50   ~ 0
-nJTRST
-Text Label 6100 7000 2    50   ~ 0
+	5700 6500 6200 6500
+Wire Wire Line
+	5700 6800 6200 6800
+Text Label 6200 6500 2    50   ~ 0
+~JTRST
+Text Label 6200 6800 2    50   ~ 0
 JTDI
-Text HLabel 5600 6900 0    50   Input ~ 0
+Text HLabel 5700 6700 0    50   Input ~ 0
 JTCK
 Wire Wire Line
-	5600 6900 6100 6900
-Text Label 6100 6900 2    50   ~ 0
+	5700 6700 6200 6700
+Text Label 6200 6700 2    50   ~ 0
 JTCK
-Text HLabel 5600 7100 0    50   Output ~ 0
+Text HLabel 5700 6900 0    50   Output ~ 0
 JTDO
 Wire Wire Line
-	5600 7100 6100 7100
-Text Label 6100 7100 2    50   ~ 0
+	5700 6900 6200 6900
+Text Label 6200 6900 2    50   ~ 0
 JTDO
 Text HLabel 1150 6150 0    50   Output ~ 0
@@
 Text Label 1550 6150 2    50   ~ 0
 NOR_RST
-Text Label 6100 7400 2    50   ~ 0
+Text Label 6200 7100 2    50   ~ 0
 USART1_TX
 Wire Wire Line
-	5600 7400 6100 7400
-Text HLabel 5600 7400 0    50   Output ~ 0
+	5700 7100 6200 7100
+Text HLabel 5700 7100 0    50   Output ~ 0
 USART_TX
-Text HLabel 5600 7300 0    50   BiDi ~ 0
-USART_CK
-Text HLabel 5600 7600 0    50   Input ~ 0
+Text HLabel 5700 7300 0    50   Input ~ 0
 USART_CTS
 Wire Wire Line
-	5600 7300 6100 7300
-Wire Wire Line
-	5600 7600 6100 7600
-Text Label 6100 7300 2    50   ~ 0
-USART1_CK
-Text Label 6100 7600 2    50   ~ 0
+	5700 7300 6200 7300
+Text Label 6200 7300 2    50   ~ 0
 USART1_CTS
-Text HLabel 5600 7500 0    50   Input ~ 0
+Text HLabel 5700 7200 0    50   Input ~ 0
 USART_RX
 Wire Wire Line
-	5600 7500 6100 7500
-Text Label 6100 7500 2    50   ~ 0
+	5700 7200 6200 7200
+Text Label 6200 7200 2    50   ~ 0
 USART1_RX
-Text HLabel 5600 7700 0    50   Output ~ 0
+Text HLabel 5700 7400 0    50   Output ~ 0
 USART_RTS
 Wire Wire Line
-	5600 7700 6100 7700
-Text Label 6100 7700 2    50   ~ 0
+	5700 7400 6200 7400
+Text Label 6200 7400 2    50   ~ 0
 USART1_RTS
 Wire Wire Line
@@
 Text Label 4100 5500 2    50   ~ 0
 LCD_ON
+Text HLabel 5700 7600 0    50   Output ~ 0
+USART_RI
+Wire Wire Line
+	5700 7600 6200 7600
+Text Label 6200 7600 2    50   ~ 0
+USART_RI
+Text HLabel 5700 7500 0    50   Input ~ 0
+USART_DSR
+Wire Wire Line
+	5700 7500 6200 7500
+Text Label 6200 7500 2    50   ~ 0
+USART_DSR
+Wire Wire Line
+	5300 4550 5300 4950
+Text Label 5300 4950 1    50   ~ 0
+USART_RI
+Wire Wire Line
+	5400 1650 5400 1250
+Wire Wire Line
+	5500 1650 5500 1250
+Text Label 5500 1250 3    50   ~ 0
+I2C1_SDA
+Text Label 5400 1250 3    50   ~ 0
+I2C1_SCL
+Wire Wire Line
+	5700 6000 6200 6000
+Wire Wire Line
+	5700 6100 6200 6100
+Text Label 6200 6100 2    50   ~ 0
+I2C1_SDA
+Text Label 6200 6000 2    50   ~ 0
+I2C1_SCL
+Text HLabel 5700 6100 0    50   BiDi ~ 0
+I2C_SDA
+Text HLabel 5700 6000 0    50   Output ~ 0
+I2C_SCL
+Wire Wire Line
+	5600 1650 5600 1250
+Wire Wire Line
+	5700 1650 5700 1250
+Text Label 5600 1250 3    50   ~ 0
+~TP_INT
+Text Label 5700 1250 3    50   ~ 0
+~TP_RST
+Wire Wire Line
+	5700 6200 6200 6200
+Wire Wire Line
+	5700 6300 6200 6300
+Text Label 6200 6300 2    50   ~ 0
+~TP_RST
+Text Label 6200 6200 2    50   ~ 0
+~TP_INT
+Text HLabel 5700 6200 0    50   Input ~ 0
+~TP_INT
+Text HLabel 5700 6300 0    50   Output ~ 0
+~TP_RST
+Wire Wire Line
+	5400 4550 5400 4950
+Text Label 5400 4950 1    50   ~ 0
+USART_DCD
+Text HLabel 5700 7700 0    50   Output ~ 0
+USART_DCD
+Wire Wire Line
+	5700 7700 6200 7700
+Text Label 6200 7700 2    50   ~ 0
+USART_DCD
+Text Notes 7000 6950 0    50   ~ 0
+Design Notes\n1. USART1/6 supports 11.25Mbit/s max\n2. All I2C support 100kHz and 400kHz modes\n3. Temperature sensor is ADC1_IN18\n4. STM32F429 : 270mA max @ 3V3 (900mW)
 Wire Bus Line
 	3650 6150 4550 6150

Commit message: R4R D1 Rev A
Parts:
- C10, C11, C12, C13, C14, C15, C16, C17, C18, C19, C20, C21, C22, C23, C24, C25, C26, C5, C6, C7, C8, C9: renamed from C?; footprint (none) -> Capacitor_SMD:C_0402_1005Metric
- SW1: renamed from SW?; footprint (none) -> Button_Switch_SMD:SW_SPST_SKQG_WithoutStem
- gave numbers to parts that had none: 1
Connections:
- net labels added: FMC_A16, FMC_A17, FMC_A18, FMC_A19, FMC_A20, FMC_A[0..20], PWROK, ~SLEEP
- net labels removed: FMC_A[0..15], LCD_B0
- wire segments 334 -> 347
- no-connect marks 0 -> 51
Other:
- note added: "Design Notes\n1. USART1/6 supports 11.25Mbit/s max\n2. All I2C support 100kHz and 400kHz modes\n3. Temperature sensor is ADC1_IN18\n4. STM32F429 : 270mA max @ 3V3 (900mW)\n5. LCD_B0 requires FMC_A20 pin. Double Flash more valuable than blue LSB"
- note removed: "Design Notes\n1. USART1/6 supports 11.25Mbit/s max\n2. All I2C support 100kHz and 400kHz modes\n3. Temperature sensor is ADC1_IN18\n4. STM32F429 : 270mA max @ 3V3 (900mW)"

Commit message: Ordered: D1 Rev A, R1 Rev B, P1 Rev B
Other:
- note added: "1. USART1/6 supports 11.25Mbit/s max\n2. All I2C support 100kHz and 400kHz modes\n3. Temperature sensor is ADC1_IN18\n4. STM32F429 : 270mA max @ 3V3 (900mW)\n5. LCD_B0 requires FMC_A20 pin. Double Flash more valuable than blue LSB"
- note removed: "Design Notes\n1. USART1/6 supports 11.25Mbit/s max\n2. All I2C support 100kHz and 400kHz modes\n3. Temperature sensor is ADC1_IN18\n4. STM32F429 : 270mA max @ 3V3 (900mW)\n5. LCD_B0 requires FMC_A20 pin. Double Flash more valuable than blue LSB"
Changed lines of the file:
@@
 $Descr A4 11693 8268
 encoding utf-8
-Sheet 4 4
-Title ""
+Sheet 3 4
+Title "D1 STM32F429"
 Date ""
 Rev ""
-Comp ""
+Comp "Puccinelli Laboratories, Inc"
 Comment1 ""
 Comment2 ""
@@
 Text Label 6200 7700 2    50   ~ 0
 USART_DCD
-Text Notes 7000 7050 0    50   ~ 0
-Design Notes\n1. USART1/6 supports 11.25Mbit/s max\n2. All I2C support 100kHz and 400kHz modes\n3. Temperature sensor is ADC1_IN18\n4. STM32F429 : 270mA max @ 3V3 (900mW)\n5. LCD_B0 requires FMC_A20 pin. Double Flash more valuable than blue LSB
+Text Notes 7000 6950 0    50   ~ 0
+1. USART1/6 supports 11.25Mbit/s max\n2. All I2C support 100kHz and 400kHz modes\n3. Temperature sensor is ADC1_IN18\n4. STM32F429 : 270mA max @ 3V3 (900mW)\n5. LCD_B0 requires FMC_A20 pin. Double Flash more valuable than blue LSB
 $Comp
 L custom-components:OSHW_logo #G3
